Commit message: fixed crazyflie2 urdf mesh reference

File: map_maker/urdf/crazyflie2.urdf.xacro (robot description, xacro)
@@ -11,5 +11,5 @@
       <origin xyz="0 0 0" rpy="1.57 0 0" />
       <geometry>
-        <mesh filename="package://crazyflie_description/meshes/crazyflie2.dae"/>
+        <mesh filename="package://map_maker/meshes/crazyflie2.dae"/>
       </geometry>
     </visual>
