Commit message: cf somewhat colored

File: map_maker/urdf/my_crazyflie.urdf.xacro (robot description, xacro)
@@ -1,4 +1,4 @@
 <?xml version="1.0"?>
-<robot xmlns:xacro="http://www.ros.org/wiki/xacro" name="my_crazyflie3">
+<robot xmlns:xacro="http://www.ros.org/wiki/xacro" name="my_crazyflie4">
   <link name="base_link">
     <inertial>
@@ -11,5 +11,5 @@
       <origin xyz="0 0 0" rpy="0 0 0" />
       <geometry>
-        <mesh filename="package://map_maker/meshes/my_crazyflie3.dae"/>
+        <mesh filename="package://map_maker/meshes/my_crazyflie4.dae"/>
       </geometry>
     </visual>
